Commit message: Created core URDF

File: description/robot.urdf.xacro (robot description, xacro)
@@ -3,4 +3,7 @@
     <!-- Include elements from robot_core.xacro -->
     <xacro:include filename="robot_core.xacro" />
+    <xacro:include filename="gazebo_control.xacro" />
+    <xacro:include filename="lidar.xacro" />
+    <xacro:include filename="camera.xacro" />
     <!-- Use elements from robot_core.xacro if needed -->
     <!-- Example: -->

File: description/robot_core.xacro (robot description, xacro)
@@ -1,5 +1,7 @@
-<?xml version="1.0"?>
 <robot xmlns:xacro="http://www.ros.org/wiki/xacro">
-      <xacro:include filename="inertial_macros.xacro" />
+  <xacro:include filename="inertial_macros.xacro" />
+  <xacro:property name="PI" value="3.1415926535897931" />
+  <xacro:property name="wheel_radius" value="0.050" />
+  <xacro:property name="wheel_width" value="0.0505" />
   <material name="white">
     <color rgba="1 1 1 1"/>
@@ -14,102 +16,179 @@
     <color rgba="0 0 0 1"/>
   </material>
-  <link name="base_link"/>
-  <joint name="chassis_joint" type="fixed">
-    <parent link="base_link"/>
-    <child link="chassis"/>
-    <origin xyz="-0.1 0 0"/>
+  <material name="red">
+    <color rgba="1 0 0 0"/>
+  </material>
+  <material name="yellow">
+    <color rgba="0.8 0.8 0.0 1.0" />
+  </material>
+  <material name="dark_grey">
+    <color rgba="0.2 0.2 0.2 1.0" />
+  </material>
+  <material name="light_grey">
+    <color rgba="0.4 0.4 0.4 1.0" />
+  </material>
+  <material name="light_purple">
+    <color rgba="0.8 0.6 1.0 1.0"/>
+  </material>
+  <link name="base_footprint" />
+  <joint name="base_link_joint" type="fixed">
+    <origin xyz="0 0 0" rpy="0 0 0" />
+    <parent link="base_footprint" />
+    <child link="base_link" />
   </joint>
-  <link name="chassis">
+  <!-- Define base link -->
+  <link name="base_link">
     <visual>
-      <origin xyz="0.15 0 0.075" rpy="0 0 0"/>
+      <origin xyz="0 0 0" rpy="0 0 0" />
       <geometry>
-        <box size="0.4 0.3 0.15"/>
+        <mesh filename="package://articubot_one/description/meshes/base_link.stl" scale="0.001 0.001 0.001"/>
       </geometry>
-      <material name="white"/>
+      <material name="light_purple" />
     </visual>
     <collision>
-      <origin xyz="0.15 0 0.075" rpy="0 0 0"/>
+      <origin xyz="0 0 0" rpy="0 0 0" />
       <geometry>
-        <box size="0.4 0.3 0.15"/>
+        <mesh filename="package://articubot_one/description/meshes/base_link.stl" scale="0.001 0.001 0.001" />
       </geometry>
-      <material name="white"/>
     </collision>
-    <xacro:inertial_box mass="0.5" x="0.3" y="0.3" z="0.15">
-        <origin xyz="0.15 0 0.075" rpy="0 0 0"/>
-    </xacro:inertial_box>
+    <inertial>
+      <origin xyz="0.0 0.0 0.12497182661389164" rpy="0 0 0"/>
+      <mass value="34.623616600117174"/>
+      <inertia ixx="0.971991" iyy="1.604575" izz="1.930029" ixy="0.0" iyz="0.0" ixz="0.0"/>
+    </inertial>
   </link>
-  <!-- LEFT WHEEL -->
-<joint name="left_wheel_joint" type="continuous">
+  <gazebo reference="base_link">
+    <material>
+      <ambient>
+        <light_purple />
+      </ambient>
+    </material>
+    <mu1>0.2</mu1>
+    <mu2>0.2</mu2>
+    <self_collide>true</self_collide>
+    <gravity>true</gravity>
+  </gazebo>
+ <joint name="upper_left_wheel_joint" type="fixed">
+  <origin xyz="-0.225 0.205 0" rpy="0 0 0" />
   <parent link="base_link"/>
-  <child link="left_wheel"/>
-  <!-- Use direct numerical value for pi/2 -->
-  <origin xyz="0 0.175 0" rpy="-1.5708 0 0"/> <!-- 1.5708 is approximately pi/2 in radians -->
-  <axis xyz="0 0 1"/>
+  <child link="upper_left_wheel" />
+  <axis xyz="0 1 0"/>
 </joint>
-  <link name="left_wheel">
-    <visual>
-      <geometry>
-        <cylinder length="0.04" radius="0.05"/>
-      </geometry>
-      <material name="blue"/>
-    </visual>
-     <collision>
-      <geometry>
-        <cylinder length="0.04" radius="0.05"/>
-      </geometry>
-      <material name="blue"/>
-    </collision>
-     <!-- ... visual and collision here ... -->
-    <xacro:inertial_cylinder mass="0.1" length="0.05" radius="0.05">
-        <origin xyz="0 0 0" rpy="0 0 0"/>
-    </xacro:inertial_cylinder>
-  </link>
-  <!-- RIGHT WHEEL -->
-  <joint name="right_wheel_joint" type="continuous">
-    <parent link="base_link"/>
-    <child link="right_wheel"/>
-    <!-- Use direct calculation of pi/2 -->
-    <origin xyz="0 -0.175 0" rpy="1.5708 0 0"/>
-    <axis xyz="0 0 -1"/>
-  </joint>
-  <link name="right_wheel">
-    <visual>
-      <geometry>
-        <cylinder length="0.04" radius="0.05"/>
-      </geometry>
-      <material name="blue"/>
-    </visual>
-     <collision>
-      <geometry>
-        <cylinder length="0.04" radius="0.05"/>
-      </geometry>
-      <material name="blue"/>
-    </collision>
-    <xacro:inertial_cylinder mass="0.1" length="0.05" radius="0.05">
-        <origin xyz="0 0 0" rpy="0 0 0"/>
-    </xacro:inertial_cylinder>
-  </link>
-  <!-- CASTER WHEEL -->
-<joint name="caster_wheel_joint" type="fixed">
-    <parent link="chassis"/>
-    <child link="caster_wheel"/>
-    <origin xyz="0.24 0 0" rpy="0 0 0"/>
+<link name="upper_left_wheel">
+  <visual>
+    <origin xyz="0 0 0" rpy="0 0 0" />
+    <geometry>
+      <mesh filename="package://articubot_one/description/meshes/mecanum_wheel_left.STL" scale="0.001 0.001 0.001"/>
+    </geometry>
+    <material name="orange" />
+  </visual>
+  <collision>
+    <origin xyz="0 0 0" rpy="${PI/2} 0 0"/>
+    <geometry>
+      <cylinder radius="${wheel_radius}" length="${wheel_width}"/>
+    </geometry>
+  </collision>
+  <inertial>
+    <origin xyz="0.0 0.0 0.0" rpy="0 0 0"/>
+    <mass value="0.3844"/>
+    <inertia
+      ixx="0.000324824" ixy="0" ixz="0"
+      iyy="0.000480000" iyz="0"
+      izz="0.000324824"/>
+  </inertial>
+</link>
+<joint name="lower_left_wheel_joint" type="fixed">
+  <origin xyz="-0.225 -0.205 0." rpy="0 0 0" />
+  <parent link="base_link"/>
+  <child link="lower_left_wheel" />
+  <axis xyz="0 1 0"/>
 </joint>
-<link name="caster_wheel">
-    <visual>
-        <geometry>
-            <sphere radius="0.05" />
-        </geometry>
-        <material name="black"/>
-    </visual>
-     <collision>
-        <geometry>
-            <sphere radius="0.05" />
-        </geometry>
-        <material name="black"/>
-    </collision>
-     <xacro:inertial_sphere mass="0.1" radius="0.05">
-        <origin xyz="0 0 0" rpy="0 0 0"/>
-    </xacro:inertial_sphere>
+<link name="lower_left_wheel">
+  <visual>
+    <origin xyz="0 0 0" rpy="0 0 0" />
+    <geometry>
+      <mesh filename="package://articubot_one/description/meshes/mecanum_wheel_left.STL" scale="0.001 0.001 0.001"/>
+    </geometry>
+    <material name="orange" />
+  </visual>
+  <collision>
+    <origin xyz="0 0 0" rpy="${PI/2} 0 0"/>
+    <geometry>
+      <cylinder radius="${wheel_radius}" length="${wheel_width}"/>
+    </geometry>
+  </collision>
+  <inertial>
+    <origin xyz="0.0 0.0 0.0" rpy="0 0 0"/>
+    <mass value="0.3844"/>
+    <inertia
+      ixx="0.000324824" ixy="0" ixz="0"
+      iyy="0.000480000" iyz="0"
+      izz="0.000324824"/>
+  </inertial>
 </link>
+<joint name="upper_right_wheel_joint" type="fixed">
+  <origin xyz="0.225 0.205 0" rpy="0 0 0" />
+  <parent link="base_link"/>
+  <child link="upper_right_wheel" />
+  <axis xyz="0 1 0"/>
+</joint>
+<link name="upper_right_wheel">
+  <visual>
+    <origin xyz="0 0 0" rpy="0 0 0" />
+    <geometry>
+      <mesh filename="package://articubot_one/description/meshes/mecanum_wheel_left.STL" scale="0.001 0.001 0.001"/>
+    </geometry>
+    <material name="orange" />
+  </visual>
+  <collision>
+    <origin xyz="0 0 0" rpy="${PI/2} 0 0"/>
+    <geometry>
+      <cylinder radius="${wheel_radius}" length="${wheel_width}"/>
+    </geometry>
+  </collision>
+  <inertial>
+    <origin xyz="0.0 0.0 0.0" rpy="0 0 0"/>
+    <mass value="0.3844"/>
+    <inertia
+      ixx="0.000324824" ixy="0" ixz="0"
+      iyy="0.000480000" iyz="0"
+      izz="0.000324824"/>
+  </inertial>
+</link>
+<joint name="lower_right_wheel_joint" type="fixed">
+  <origin xyz="0.225 -0.205 0" rpy="0 0 0" />
+  <parent link="base_link"/>
+  <child link="lower_right_wheel" />
+  <axis xyz="0 1 0"/>
+</joint>
+<link name="lower_right_wheel">
+  <visual>
+    <origin xyz="0 0 0" rpy="0 0 0" />
+    <geometry>
+      <mesh filename="package://articubot_one/description/meshes/mecanum_wheel_left.STL" scale="0.001 0.001 0.001"/>
+    </geometry>
+    <material name="orange" />
+  </visual>
+  <collision>
+    <origin xyz="0 0 0" rpy="${PI/2} 0 0"/>
+    <geometry>
+      <cylinder radius="${wheel_radius}" length="${wheel_width}"/>
+    </geometry>
+  </collision>
+  <inertial>
+    <origin xyz="0.0 0.0 0.0" rpy="0 0 0"/>
+    <mass value="0.3844"/>
+    <inertia
+      ixx="0.000324824" ixy="0" ixz="0"
+      iyy="0.000480000" iyz="0"
+      izz="0.000324824"/>
+  </inertial>
+</link>
+  <gazebo reference="lower_right_wheel">
+    <material>
+      <ambient>
+        <yellow />
+      </ambient>
+    </material>
+  </gazebo>
 </robot>
