Commit message: spawn the robot on gazebo with editing the core URDF

File: description/camera.xacro (robot description, xacro)
@@ -1,57 +1,61 @@
 <?xml version="1.0"?>
 <robot xmlns:xacro="http://www.ros.org/wiki/xacro">
-    <link name="camera_link">
-        <inertial>
-            <origin xyz="-5.607908532515647e-05 -1.1159512353752273e-14 0.11972685138201877" rpy="0 0 0"/>
-            <mass value="0.24695182299262655"/>
-            <inertia ixx="0.000829" iyy="0.000765" izz="0.000109" ixy="0.0" iyz="0.0" ixz="1e-06"/>
-        </inertial>
-        <visual>
-            <origin xyz="-0.0 -0.0 -0.25" rpy="0 0 0"/>
-            <geometry>
-                <mesh filename="package://articubot_one/description/meshes/camera_link.stl" scale="0.001 0.001 0.001"/>
-            </geometry>
-            <material name="dark_grey"/>
-        </visual>
-        <collision>
-            <origin xyz="-0.0 -0.0 -0.25" rpy="0 0 0"/>
-            <geometry>
-                <mesh filename="package://articubot_one/description/meshes/camera_link.stl" scale="0.001 0.001 0.001"/>
-            </geometry>
-        </collision>
-    </link>
-    <joint name="camera_joint" type="fixed">
-        <parent link="base_link"/>
-        <child link="camera_link"/>
-        <origin xyz="0.0 0.0 0.25" rpy="0 0 0"/>
-    </joint>
-    <link name="camera_link_optical"></link>
-    <joint name="camera_optical_joint" type="fixed">
-        <parent link="camera_link"/>
-        <child link="camera_link_optical"/>
-        <origin xyz="0 0 0" rpy="0 ${-pi/2} ${-pi/2}"/>
-    </joint>
-    <gazebo reference="camera_link">
-        <material>Gazebo/Red</material>
-        <sensor name="camera" type="camera">
-            <pose>0 0 0 0 0 0</pose>
-            <visualize>true</visualize>
-            <update_rate>10</update_rate>
-            <camera>
-                <horizontal_fov>1.089</horizontal_fov>
-                <image>
-                    <format>R8G8B8</format>
-                    <width>640</width>
-                    <height>480</height>
-                </image>
-                <clip>
-                    <near>0.05</near>
-                    <far>8.0</far>
-                </clip>
-            </camera>
-            <plugin name="camera_controller" filename="libgazebo_ros_camera.so">
-                <frame_name>camera_link_optical</frame_name>
-            </plugin>
-        </sensor>
-    </gazebo>
+  <link name="camera_link">
+      <xacro:inertial_cylinder mass="0.24695182299262655" radius="0.05" length="0.24">
+        <origin xyz="0.0 0.0 -0.46" rpy="0 0 0"/>
+      </xacro:inertial_cylinder>
+    <visual>
+      <origin xyz="0.0 0.0 -0.46" rpy="0 0 0"/>
+      <geometry>
+        <mesh filename="$(find articubot_one)/description/meshes/camera_link.stl" scale="0.001 0.001 0.001"/>
+      </geometry>
+      <material name="dark_grey"/>
+    </visual>
+    <collision>
+      <origin xyz="0.0 0.0 -0.03" rpy="0 0 0"/>
+      <geometry>
+        <cylinder radius="0.05" length="0.24"/>
+      </geometry>
+    </collision>
+  </link>
+  <joint name="camera_joint" type="fixed">
+    <parent link="base_link"/>
+    <child link="camera_link"/>
+    <origin xyz="0.0 0.0 0.45" rpy="0 0 0"/>
+  </joint>
+  <link name="camera_link_optical">
+    <inertial>
+      <origin xyz="0 0 0" rpy="0 0 0"/>
+      <mass value="0.01"/>
+      <inertia ixx="0.00001" iyy="0.00001" izz="0.00001" ixy="0.0" iyz="0.0" ixz="0.0"/>
+    </inertial>
+  </link>
+  <joint name="camera_optical_joint" type="fixed">
+    <parent link="camera_link"/>
+    <child link="camera_link_optical"/>
+    <origin xyz="0 0 0" rpy="0 ${-PI/2} ${-PI/2}"/>
+  </joint>
+  <gazebo reference="camera_link">
+    <material>Gazebo/Grey</material>
+    <sensor name="camera" type="camera">
+      <pose>0 0 0 0 0 0</pose>
+      <visualize>true</visualize>
+      <update_rate>10</update_rate>
+      <camera>
+        <horizontal_fov>1.089</horizontal_fov>
+        <image>
+          <format>R8G8B8</format>
+          <width>640</width>
+          <height>480</height>
+        </image>
+        <clip>
+          <near>0.05</near>
+          <far>8.0</far>
+        </clip>
+      </camera>
+      <plugin name="camera_controller" filename="libgazebo_ros_camera.so">
+        <frame_name>camera_link_optical</frame_name>
+      </plugin>
+    </sensor>
+  </gazebo>
 </robot>

File: description/lidar.xacro (robot description, xacro)
@@ -1,33 +1,31 @@
 <?xml version="1.0"?>
 <robot xmlns:xacro="http://www.ros.org/wiki/xacro">
+ <xacro:include filename="inertial_macros.xacro" />
     <joint name="laser_joint" type="fixed">
         <parent link="base_link"/>
         <child link="laser_frame"/>
-        <origin xyz="0.2 -0.1 0.25" rpy="0 0 0"/>
+        <origin xyz="0.15 0 0.3" rpy="0 0 0"/>
     </joint>
     <link name="laser_frame">
-        <inertial>
-            <origin xyz="-0.09451642096837788 0.1 0.011806551131625875" rpy="0 0 0"/>
-            <mass value="0.058519310420852316"/>
-            <inertia ixx="1e-05" iyy="1.8e-05" izz="2e-05" ixy="0.0" iyz="-0.0" ixz="2e-06"/>
-        </inertial>
-        <visual>
-            <origin xyz="-0.2 0.1 -0.25" rpy="0 0 0"/>
+      <xacro:inertial_cylinder mass="0.058519310420852316" radius="0.05" length="0.05">
+        <origin xyz="-0.11 0 -0.3" rpy="0 0 0"/>
+      </xacro:inertial_cylinder>
+       <visual>
+            <origin xyz="-0.11 0 -0.3" rpy="0 0 0"/>
             <geometry>
-                <mesh filename="package://articubot_one/description/meshes/lidar_1.stl" scale="0.001 0.001 0.001"/>
+                <mesh filename="$(find articubot_one)/description/meshes/lidar_1.stl" scale="0.001 0.001 0.001"/>
             </geometry>
-            <material name="bleu"/> <!-- Set material to bleu (blue) -->
         </visual>
         <collision>
-            <origin xyz="-0.2 0.1 -0.25" rpy="0 0 0"/>
-            <geometry>
-                <mesh filename="package://articubot_one/description/meshes/lidar_1.stl" scale="0.001 0.001 0.001"/>
-            </geometry>
+               <origin xyz="0 0 0.025" rpy="0 0 0"/>
+               <geometry>
+               <cylinder radius="0.05" length="0.05"/>
+               </geometry>
         </collision>
     </link>
     <gazebo reference="laser_frame">
-        <material>Gazebo/bleu</material>
+         <material>Gazebo/Orange</material>
         <sensor name="laser" type="ray">
-            <pose> 0 0 0 0 0 0 </pose>
+            <pose>0 0 0 0 0 0</pose>
             <visualize>true</visualize>
             <update_rate>10</update_rate>
@@ -47,4 +45,6 @@
             <plugin name="laser_controller" filename="libgazebo_ros_ray_sensor.so">
                 <ros>
+                    <argument>--ros-args</argument>
+                    <argument>--remap</argument>
                     <argument>~/out:=scan</argument>
                 </ros>

File: description/robot.urdf.xacro (robot description, xacro)
@@ -3,5 +3,4 @@
     <!-- Include elements from robot_core.xacro -->
     <xacro:include filename="robot_core.xacro" />
-    <xacro:include filename="gazebo_control.xacro" />
     <xacro:include filename="lidar.xacro" />
     <xacro:include filename="camera.xacro" />

File: description/robot_core.xacro (robot description, xacro)
@@ -1,12 +1,10 @@
+<?xml version="1.0"?>
 <robot xmlns:xacro="http://www.ros.org/wiki/xacro">
+  <xacro:property name="PI" value="3.1415926535897931" />
   <xacro:include filename="inertial_macros.xacro" />
-  <xacro:property name="PI" value="3.1415926535897931" />
-  <xacro:property name="wheel_radius" value="0.050" />
-  <xacro:property name="wheel_width" value="0.0505" />
+  <xacro:include filename="$(find articubot_one)/description/mecanum_wheel/mecanum_wheel.urdf.xacro"/>
+  <!-- Material Definitions -->
   <material name="white">
     <color rgba="1 1 1 1"/>
-  </material>
-  <material name="orange">
-    <color rgba="1 0.3 0.1 1"/>
   </material>
   <material name="blue">
@@ -17,14 +15,14 @@
   </material>
   <material name="red">
-    <color rgba="1 0 0 0"/>
+    <color rgba="1 0 0 1"/>
   </material>
   <material name="yellow">
-    <color rgba="0.8 0.8 0.0 1.0" />
+    <color rgba="0.8 0.8 0.0 1.0"/>
   </material>
   <material name="dark_grey">
-    <color rgba="0.2 0.2 0.2 1.0" />
+    <color rgba="0.2 0.2 0.2 1.0"/>
   </material>
   <material name="light_grey">
-    <color rgba="0.4 0.4 0.4 1.0" />
+    <color rgba="0.4 0.4 0.4 1.0"/>
   </material>
   <material name="light_purple">
@@ -33,5 +31,5 @@
   <link name="base_footprint" />
   <joint name="base_link_joint" type="fixed">
-    <origin xyz="0 0 0" rpy="0 0 0" />
+    <origin xyz="0 0 0.04" rpy="0 0 0" />
     <parent link="base_footprint" />
     <child link="base_link" />
@@ -39,156 +37,58 @@
   <!-- Define base link -->
   <link name="base_link">
+    <xacro:inertial_box mass="4.0990470908566525" x="0.7" y="0.5" z="0.3">
+              <origin xyz="0 0 0" rpy="0 0 0"/>
+    </xacro:inertial_box>
     <visual>
-      <origin xyz="0 0 0" rpy="0 0 0" />
+      <origin xyz="0 0 0" rpy="0 0 0"/>
       <geometry>
-        <mesh filename="package://articubot_one/description/meshes/base_link.stl" scale="0.001 0.001 0.001"/>
+        <mesh filename="$(find articubot_one)/description/meshes/base_link.stl" scale="0.001 0.001 0.001"/>
       </geometry>
-      <material name="light_purple" />
+      <material name="light_purple"/>
     </visual>
     <collision>
-      <origin xyz="0 0 0" rpy="0 0 0" />
+      <origin xyz="0 0 0.15" rpy="0 0 0"/>
       <geometry>
-        <mesh filename="package://articubot_one/description/meshes/base_link.stl" scale="0.001 0.001 0.001" />
+        <box size="0.7 0.5 0.3"/>
       </geometry>
     </collision>
-    <inertial>
-      <origin xyz="0.0 0.0 0.12497182661389164" rpy="0 0 0"/>
-      <mass value="34.623616600117174"/>
-      <inertia ixx="0.971991" iyy="1.604575" izz="1.930029" ixy="0.0" iyz="0.0" ixz="0.0"/>
-    </inertial>
   </link>
+  <!-- Upper Left Wheel -->
+  <xacro:wheel_v0 prefix="upper" parent="base_link">
+    <origin xyz="0.2 0.275 0.01" rpy="0 0 ${PI}"/>
+    <axis xyz="0 1 0"/>
+  </xacro:wheel_v0>
+  <!-- Lower Left Wheel -->
+  <xacro:wheel_v0 prefix="lower" parent="base_link">
+    <origin xyz="-0.2 0.275 0.01" rpy="0 0 ${PI}"/>
+    <axis xyz="0 1 0"/>
+  </xacro:wheel_v0>
+  <!-- Upper Right Wheel -->
+  <xacro:wheel_v1 prefix="upper" parent="base_link">
+    <origin xyz="0.2 -0.275 0.01" rpy="0 0 0"/>
+    <axis xyz="0 -1 0"/>
+  </xacro:wheel_v1>
+  <!-- Lower Right Wheel -->
+  <xacro:wheel_v1 prefix="lower" parent="base_link">
+    <origin xyz="-0.2 -0.275 0.01" rpy="0 0 0"/>
+    <axis xyz="0 -1 0"/>
+  </xacro:wheel_v1>
+  <!-- Transmissions -->
+  <xacro:wheel_trans_v0 prefix="upper_right"/>
+  <xacro:wheel_trans_v0 prefix="upper_left"/>
+  <xacro:wheel_trans_v0 prefix="lower_right"/>
+  <xacro:wheel_trans_v0 prefix="lower_left"/>
+  <!-- Gazebo -->
   <gazebo reference="base_link">
-    <material>
-      <ambient>
-        <light_purple />
-      </ambient>
-    </material>
+    <material>Gazebo/Purple</material>
     <mu1>0.2</mu1>
     <mu2>0.2</mu2>
-    <self_collide>true</self_collide>
+    <self_collide>false</self_collide>
     <gravity>true</gravity>
   </gazebo>
- <joint name="upper_left_wheel_joint" type="fixed">
-  <origin xyz="-0.225 0.205 0" rpy="0 0 0" />
-  <parent link="base_link"/>
-  <child link="upper_left_wheel" />
-  <axis xyz="0 1 0"/>
-</joint>
-<link name="upper_left_wheel">
-  <visual>
-    <origin xyz="0 0 0" rpy="0 0 0" />
-    <geometry>
-      <mesh filename="package://articubot_one/description/meshes/mecanum_wheel_left.STL" scale="0.001 0.001 0.001"/>
-    </geometry>
-    <material name="orange" />
-  </visual>
-  <collision>
-    <origin xyz="0 0 0" rpy="${PI/2} 0 0"/>
-    <geometry>
-      <cylinder radius="${wheel_radius}" length="${wheel_width}"/>
-    </geometry>
-  </collision>
-  <inertial>
-    <origin xyz="0.0 0.0 0.0" rpy="0 0 0"/>
-    <mass value="0.3844"/>
-    <inertia
-      ixx="0.000324824" ixy="0" ixz="0"
-      iyy="0.000480000" iyz="0"
-      izz="0.000324824"/>
-  </inertial>
-</link>
-<joint name="lower_left_wheel_joint" type="fixed">
-  <origin xyz="-0.225 -0.205 0." rpy="0 0 0" />
-  <parent link="base_link"/>
-  <child link="lower_left_wheel" />
-  <axis xyz="0 1 0"/>
-</joint>
-<link name="lower_left_wheel">
-  <visual>
-    <origin xyz="0 0 0" rpy="0 0 0" />
-    <geometry>
-      <mesh filename="package://articubot_one/description/meshes/mecanum_wheel_left.STL" scale="0.001 0.001 0.001"/>
-    </geometry>
-    <material name="orange" />
-  </visual>
-  <collision>
-    <origin xyz="0 0 0" rpy="${PI/2} 0 0"/>
-    <geometry>
-      <cylinder radius="${wheel_radius}" length="${wheel_width}"/>
-    </geometry>
-  </collision>
-  <inertial>
-    <origin xyz="0.0 0.0 0.0" rpy="0 0 0"/>
-    <mass value="0.3844"/>
-    <inertia
-      ixx="0.000324824" ixy="0" ixz="0"
-      iyy="0.000480000" iyz="0"
-      izz="0.000324824"/>
-  </inertial>
-</link>
-<joint name="upper_right_wheel_joint" type="fixed">
-  <origin xyz="0.225 0.205 0" rpy="0 0 0" />
-  <parent link="base_link"/>
-  <child link="upper_right_wheel" />
-  <axis xyz="0 1 0"/>
-</joint>
-<link name="upper_right_wheel">
-  <visual>
-    <origin xyz="0 0 0" rpy="0 0 0" />
-    <geometry>
-      <mesh filename="package://articubot_one/description/meshes/mecanum_wheel_left.STL" scale="0.001 0.001 0.001"/>
-    </geometry>
-    <material name="orange" />
-  </visual>
-  <collision>
-    <origin xyz="0 0 0" rpy="${PI/2} 0 0"/>
-    <geometry>
-      <cylinder radius="${wheel_radius}" length="${wheel_width}"/>
-    </geometry>
-  </collision>
-  <inertial>
-    <origin xyz="0.0 0.0 0.0" rpy="0 0 0"/>
-    <mass value="0.3844"/>
-    <inertia
-      ixx="0.000324824" ixy="0" ixz="0"
-      iyy="0.000480000" iyz="0"
-      izz="0.000324824"/>
-  </inertial>
-</link>
-<joint name="lower_right_wheel_joint" type="fixed">
-  <origin xyz="0.225 -0.205 0" rpy="0 0 0" />
-  <parent link="base_link"/>
-  <child link="lower_right_wheel" />
-  <axis xyz="0 1 0"/>
-</joint>
-<link name="lower_right_wheel">
-  <visual>
-    <origin xyz="0 0 0" rpy="0 0 0" />
-    <geometry>
-      <mesh filename="package://articubot_one/description/meshes/mecanum_wheel_left.STL" scale="0.001 0.001 0.001"/>
-    </geometry>
-    <material name="orange" />
-  </visual>
-  <collision>
-    <origin xyz="0 0 0" rpy="${PI/2} 0 0"/>
-    <geometry>
-      <cylinder radius="${wheel_radius}" length="${wheel_width}"/>
-    </geometry>
-  </collision>
-  <inertial>
-    <origin xyz="0.0 0.0 0.0" rpy="0 0 0"/>
-    <mass value="0.3844"/>
-    <inertia
-      ixx="0.000324824" ixy="0" ixz="0"
-      iyy="0.000480000" iyz="0"
-      izz="0.000324824"/>
-  </inertial>
-</link>
-  <gazebo reference="lower_right_wheel">
-    <material>
-      <ambient>
-        <yellow />
-      </ambient>
-    </material>
-  </gazebo>
+  <!-- Wheel Gazebo -->
+  <xacro:wheel_gazebo_v0 prefix="upper_right"/>
+  <xacro:wheel_gazebo_v0 prefix="upper_left"/>
+  <xacro:wheel_gazebo_v0 prefix="lower_right"/>
+  <xacro:wheel_gazebo_v0 prefix="lower_left"/>
 </robot>

Commit message: visualisation of the robot in odom fixed frame by adding the joint state publisher

File: description/camera.xacro (robot description, xacro)
@@ -8,5 +8,5 @@
       <origin xyz="0.0 0.0 -0.46" rpy="0 0 0"/>
       <geometry>
-        <mesh filename="$(find articubot_one)/description/meshes/camera_link.stl" scale="0.001 0.001 0.001"/>
+        <mesh filename="file://$(find articubot_one)/description/meshes/camera_link.stl" scale="0.001 0.001 0.001"/>
       </geometry>
       <material name="dark_grey"/>

File: description/lidar.xacro (robot description, xacro)
@@ -7,5 +7,5 @@
         <parent link="base_link"/>
         <child link="laser_frame"/>
-        <origin xyz="0.15 0 0.3" rpy="0 0 0"/>
+        <origin xyz="0.15 0 0.33" rpy="0 0 0"/>
     </joint>
     <!-- Define the laser frame link -->
@@ -17,7 +17,7 @@
         </inertial>
         <visual>
-            <origin xyz="-0.11 0 -0.3" rpy="0 0 0"/>
+            <origin xyz="-0.11 0 -0.33" rpy="0 0 0"/>
             <geometry>
-                <mesh filename="$(find articubot_one)/description/meshes/lidar_1.stl" scale="0.001 0.001 0.001"/>
+                <mesh filename="file://$(find articubot_one)/description/meshes/lidar_1.stl" scale="0.001 0.001 0.001"/>
             </geometry>
         </visual>

File: description/mecanum_wheel/mecanum_wheel.urdf.xacro (robot description, xacro)
@@ -24,5 +24,5 @@
         <origin xyz="0 0 0" rpy="0 0 0" />
         <geometry>
-          <mesh filename="$(find articubot_one)/description/meshes/mecanum_wheel_left.STL" scale="0.001 0.001 0.001"/>
+          <mesh filename="file://$(find articubot_one)/description/meshes/mecanum_wheel_left.STL" scale="0.001 0.001 0.001"/>
         </geometry>
         <material name="orange" />
@@ -71,5 +71,5 @@
         <origin xyz="0 0 0" rpy="0 0 0" />
         <geometry>
-          <mesh filename="$(find articubot_one)/description/meshes/mecanum_wheel_right.STL" scale="0.001 0.001 0.001"/>
+          <mesh filename="file://$(find articubot_one)/description/meshes/mecanum_wheel_right.STL" scale="0.001 0.001 0.001"/>
         </geometry>
         <material name="orange" />

File: description/robot_core.xacro (robot description, xacro)
@@ -43,5 +43,5 @@
       <origin xyz="0 0 0" rpy="0 0 0"/>
       <geometry>
-        <mesh filename="$(find articubot_one)/description/meshes/base_link.stl" scale="0.001 0.001 0.001"/>
+        <mesh filename="file://$(find articubot_one)/description/meshes/base_link.stl" scale="0.001 0.001 0.001"/>
       </geometry>
       <material name="light_purple"/>
