Commit message: add lidar and launch the robot in my world

File: description/lidar.xacro (robot description, xacro)
@@ -1,5 +1,7 @@
 <?xml version="1.0"?>
 <robot xmlns:xacro="http://www.ros.org/wiki/xacro">
- <xacro:include filename="inertial_macros.xacro" />
+    <!-- Including external xacro file for inertial macros -->
+    <xacro:include filename="inertial_macros.xacro" />
+    <!-- Define a fixed joint for the laser -->
     <joint name="laser_joint" type="fixed">
         <parent link="base_link"/>
@@ -7,9 +9,12 @@
         <origin xyz="0.15 0 0.3" rpy="0 0 0"/>
     </joint>
+    <!-- Define the laser frame link -->
     <link name="laser_frame">
-      <xacro:inertial_cylinder mass="0.058519310420852316" radius="0.05" length="0.05">
-        <origin xyz="-0.11 0 -0.3" rpy="0 0 0"/>
-      </xacro:inertial_cylinder>
-       <visual>
+        <inertial>
+            <origin xyz="-0.11 0 -0.3" rpy="0 0 0"/>
+            <mass value="0.058519310420852316"/>
+            <inertia ixx="0.0001" ixy="0.0" ixz="0.0" iyy="0.0001" iyz="0.0" izz="0.0001"/>
+        </inertial>
+        <visual>
             <origin xyz="-0.11 0 -0.3" rpy="0 0 0"/>
             <geometry>
@@ -18,14 +23,14 @@
         </visual>
         <collision>
-               <origin xyz="0 0 0.025" rpy="0 0 0"/>
-               <geometry>
-               <cylinder radius="0.05" length="0.05"/>
-               </geometry>
+            <origin xyz="0 0 0.025" rpy="0 0 0"/>
+            <geometry>
+                <cylinder radius="0.05" length="0.05"/>
+            </geometry>
         </collision>
     </link>
     <gazebo reference="laser_frame">
-         <material>Gazebo/Orange</material>
+        <material>Gazebo/Red</material>
         <sensor name="laser" type="ray">
-            <pose>0 0 0 0 0 0</pose>
+            <pose>0 0 0.01 0 0 0</pose>
             <visualize>true</visualize>
             <update_rate>10</update_rate>
@@ -45,7 +50,6 @@
             <plugin name="laser_controller" filename="libgazebo_ros_ray_sensor.so">
                 <ros>
-                    <argument>--ros-args</argument>
-                    <argument>--remap</argument>
-                    <argument>~/out:=scan</argument>
+                    <namespace>/</namespace>
+                    <remapping>out:=/scan</remapping>
                 </ros>
                 <output_type>sensor_msgs/LaserScan</output_type>

File: description/mecanum_wheel/mecanum_wheel.urdf.xacro (robot description, xacro)
@@ -17,5 +17,5 @@
       <parent link="${parent}"/>
       <child link="${prefix}_left_wheel_link"/>
-      <limit effort="100" velocity="100"/>
+      <limit effort="100" velocity="300"/>
       <xacro:insert_block name="joint_axis"/>
     </joint>
@@ -40,6 +40,6 @@
         <friction>
           <ode>
-            <mu>1.2</mu>
-            <mu2>1.2</mu2>
+            <mu>0.9</mu>
+            <mu2>0.9</mu2>
             <kp>1e15</kp>
             <kd>1e13</kd>
@@ -64,5 +64,5 @@
       <parent link="${parent}"/>
       <child link="${prefix}_right_wheel_link"/>
-      <limit effort="100" velocity="100"/>
+      <limit effort="100" velocity="300"/>
       <xacro:insert_block name="joint_axis"/>
     </joint>
@@ -87,6 +87,6 @@
         <friction>
           <ode>
-            <mu>1.2</mu>
-            <mu2>1.2</mu2>
+            <mu>0.9</mu>
+            <mu2>0.9</mu2>
             <kp>1e15</kp>
             <kd>1e13</kd>

File: description/robot_core.xacro (robot description, xacro)
@@ -81,7 +81,5 @@
   <!-- Gazebo -->
   <gazebo reference="base_link">
-    <material>Gazebo/Purple</material>
-    <mu1>0.2</mu1>
-    <mu2>0.2</mu2>
+    <material>Gazebo/Green</material>
     <self_collide>false</self_collide>
     <gravity>true</gravity>

Commit message: add a launch file for outdoor world and take the two maps

File: description/lidar.xacro (robot description, xacro)
@@ -34,5 +34,5 @@
             <pose>0 0 0.01 0 0 0</pose>
             <visualize>true</visualize>
-            <update_rate>10</update_rate>
+            <update_rate>100</update_rate>
             <ray>
                 <scan>

File: description/robot_core.xacro (robot description, xacro)
@@ -29,6 +29,7 @@
     <color rgba="0.8 0.6 1.0 1.0"/>
   </material>
-  <link name="base_footprint" />
-  <joint name="base_link_joint" type="fixed">
+  <link name="base_footprint">
+  </link>
+  <joint name="base_footprint_to_base_link" type="fixed">
     <origin xyz="0 0 0.04" rpy="0 0 0" />
     <parent link="base_footprint" />
@@ -38,5 +39,5 @@
   <link name="base_link">
     <xacro:inertial_box mass="4.0990470908566525" x="0.7" y="0.5" z="0.3">
-              <origin xyz="0 0 0" rpy="0 0 0"/>
+      <origin xyz="0 0 0" rpy="0 0 0"/>
     </xacro:inertial_box>
     <visual>
